File: hardware/teensy-touch.kicad_pcb (KiCad board)
At the start: 2 copper layers, 66 x 60 mm, 15 parts, among them J1 TEENSY-LC, J2 OLED_128x64

Commit message: connect GND pin for OLED to GND plane
Routing:
- net /GND: track 0.00 -> 4.25 mm, vias 0 -> 1
Changed lines of the file:
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@@
   (general
     (links 18)
-    (no_connects 1)
-    (area 106.553 83.439 229.235 148.463)
+    (no_connects 0)
+    (area 106.579999 83.465999 174.18502 148.2064)
     (thickness 1.6)
     (drawings 25)
-    (tracks 245)
+    (tracks 248)
     (zones 0)
     (modules 15)
@@
     (34 B.Paste user hide)
     (35 F.Paste user hide)
-    (36 B.SilkS user)
-    (37 F.SilkS user)
-    (38 B.Mask user)
-    (39 F.Mask user)
+    (36 B.SilkS user hide)
+    (37 F.SilkS user hide)
+    (38 B.Mask user hide)
+    (39 F.Mask user hide)
     (40 Dwgs.User user hide)
     (41 Cmts.User user hide)
-    (42 Eco1.User user)
+    (42 Eco1.User user hide)
     (43 Eco2.User user hide)
     (44 Edge.Cuts user)
@@
   )
   (setup
-    (last_trace_width 0.1524)
+    (last_trace_width 0.508)
+    (user_trace_width 0.254)
+    (user_trace_width 0.508)
+    (user_trace_width 2.54)
     (trace_clearance 0.1524)
     (zone_clearance 0.508)
@@
     (via_min_size 0.6858)
     (via_min_drill 0.3302)
+    (user_via 0.762 0.508)
     (uvia_size 0.3)
     (uvia_drill 0.1)
@@
   (segment (start 161.036 124.841) (end 157.099 128.778) (width 0.508) (layer B.Cu) (net 17) (status 80000))
   (segment (start 157.099 128.778) (end 156.591 128.778) (width 0.508) (layer B.Cu) (net 17) (status 80000))
+  (segment (start 168.91 108.077) (end 168.91 105.537) (width 0.508) (layer F.Cu) (net 18))
+  (via (at 170.1165 104.3305) (size 0.6858) (drill 0.3302) (layers F.Cu B.Cu) (net 18))
+  (segment (start 168.91 105.537) (end 170.1165 104.3305) (width 0.508) (layer F.Cu) (net 18))
   (segment (start 156.591 100.838) (end 159.639 103.886) (width 0.508) (layer F.Cu) (net 19) (status 80000))
   (segment (start 159.639 103.886) (end 159.639 104.013) (width 0.508) (layer F.Cu) (net 19) (status 80000))
